File: Gotek.kicad_pcb (KiCad board)
At the start: 2 copper layers, 111.6 x 59.4 mm, 77 parts, among them J10 Conn_01x04_Pin, J3 Conn_01x03_Pin, J4 Conn_01x02_Pin, J5 Conn_01x02, J7 OLED, J8 RotaryEncoder, P1 2005280260, P3 USB_A, Q1 PMBT2222A,215, Q2 PMBT2222A,215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

Commit message: Add files via upload
Removed L3 Green LED and changed R21 to 12K to reduce it's brightness. Also increased the pad sizes for the diode D1D to make it easier to hand solder. Minor changes to silk screen.
Parts:
- R21: value 1K -> 12K
Other:
- board text added: "SEL"
- board text removed: "+5V"
- board text removed: "2"
- board text removed: "GND"
Changed lines of the file:
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@@
 		(tags "resistor handsolder")
 		(property "Reference" "PU5"
-			(at -3.683 -0.1778 0)
+			(at -4.133 0.2113 0)
 			(layer "F.SilkS")
 			(effects
@@
 		(sheetname "Root")
 		(sheetfile "Gotek.kicad_sch")
-		(attr through_hole dnp)
+		(attr through_hole)
 		(fp_line
 			(start -0.79 -1.399)
@@
 		(tags "capacitor handsolder")
 		(property "Reference" "C20"
-			(at -1.258025 -1.8669 0)
+			(at -0.1082 -1.9114 0)
 			(layer "F.SilkS")
 			(effects
@@
 		(tags "resistor handsolder")
 		(property "Reference" "PU13"
-			(at 4.16535 1.330325 0)
+			(at 0.1712 8.2772 0)
 			(layer "F.SilkS")
 			(effects
@@
 		(tags "Power Supply")
 		(property "Reference" "Q3"
-			(at 3.02895 0.815975 0)
+			(at -0.0571 10.0362 0)
 			(layer "F.SilkS")
 			(effects
@@
 		(tags "resistor handsolder")
 		(property "Reference" "PU9"
-			(at -3.965575 0.10795 0)
+			(at -3.828 0.2844 0)
 			(layer "F.SilkS")
 			(effects
@@
 		(tags "Through hole angled pin header THT 1x02 2.54mm single row")
 		(property "Reference" "JE1"
-			(at 4.385 -2.27 0)
+			(at -1.9722 0.9808 0)
 			(layer "F.SilkS")
 			(effects
@@
 		(tags "resistor handsolder")
 		(property "Reference" "RN2"
-			(at -0.9708 -5.991225 0)
+			(at -0.1326 -7.2295 0)
 			(layer "F.SilkS")
 			(effects
@@
 		(tags "resistor handsolder")
 		(property "Reference" "PU8"
-			(at 3.736725 1.53035 0)
+			(at -0.286 11.8459 0)
 			(layer "F.SilkS")
 			(effects
@@
 		(tags "resistor handsolder")
 		(property "Reference" "RN1"
-			(at -0.92635 -4.340225 0)
+			(at -0.1326 -5.9087 0)
 			(layer "F.SilkS")
 			(effects
@@
 		(tags "Power Supply")
 		(property "Reference" "Q2"
-			(at 3.051175 -1.565275 0)
+			(at 0.0191 7.82 0)
 			(layer "F.SilkS")
 			(effects
@@
 		(pad "1" smd rect
 			(at -1.15 0 270)
-			(size 0.42 0.82)
+			(size 1 1)
 			(layers "F.Cu" "F.Paste" "F.Mask")
 			(net 7 "Net-(DID1-K)")
@@
 		(pad "2" smd rect
 			(at 1.15 0 270)
-			(size 0.42 0.82)
+			(size 1 1)
 			(layers "F.Cu" "F.Paste" "F.Mask")
 			(net 56 "Net-(DID1-A)")
@@
 		(tags "resistor handsolder")
 		(property "Reference" "RN3"
-			(at -0.9708 -7.6073 0)
+			(at -0.031 -8.6931 0)
 			(layer "F.SilkS")
 			(effects
@@
 		(tags "Through hole angled pin header THT 1x02 2.54mm single row")
 		(property "Reference" "JD1"
-			(at 4.385 -2.27 0)
+			(at -2.2008 1.3002 0)
 			(layer "F.SilkS")
 			(effects
@@
 		(tags "resistor handsolder")
 		(property "Reference" "PU6"
-			(at 3.781175 0.5842 0)
+			(at -0.286 13.3731 0)
 			(layer "F.SilkS")
 			(effects
@@
 		(tags "resistor handsolder")
 		(property "Reference" "PU10"
-			(at 3.97485 0.6096 0)
+			(at 0.19 9.9663 0)
 			(layer "F.SilkS")
 			(effects
@@
 		(tags "Power Supply")
 		(property "Reference" "Q1"
-			(at 3.048 -4.098925 0)
+			(at 0.0635 5.4165 0)
 			(layer "F.SilkS")
 			(effects
@@
 			)
 		)
-		(property "Value" "1K"
+		(property "Value" "12K"
 			(at 0 1.65 0)
 			(layer "F.Fab")
@@
 		(tags "resistor handsolder")
 		(property "Reference" "PU4"
-			(at -3.82245 -0.40005 0)
+			(at -0.286 15.113 0)
 			(layer "F.SilkS")
 			(effects
@@
 		(tags "resistor handsolder")
 		(property "Reference" "PU7"
-			(at -3.62585 -0.06985 0)
+			(at -4.108 0.5383 0)
 			(layer "F.SilkS")
 			(effects
@@
 		(tags "Through hole angled pin header THT 1x03 2.54mm single row")
 		(property "Reference" "MO1"
-			(at 4.385 -2.27 0)
+			(at -2.4294 4.4106 0)
 			(layer "F.SilkS")
 			(effects
@@
 	)
 	(gr_line
+		(start 178.2318 58.0136)
+		(end 160.8328 58.0136)
+		(stroke
+			(width 0.1)
+			(type default)
+		)
+		(layer "F.SilkS")
+	)
+	(gr_line
+		(start 149.5298 105.3084)
+		(end 139.8524 105.3084)
+		(stroke
+			(width 0.1)
+			(type default)
+		)
+		(layer "F.SilkS")
+	)
+	(gr_line
+		(start 144.66394 103.2764)
+		(end 144.66394 110.2614)
+		(stroke
+			(width 0.1)
+			(type default)
+		)
+		(layer "F.SilkS")
+	)
+	(gr_line
+		(start 149.479 107.0102)
+		(end 139.7762 107.0102)
+		(stroke
+			(width 0.1)
+			(type default)
+		)
+		(layer "F.SilkS")
+	)
+	(gr_line
+		(start 139.8016 105.3084)
+		(end 149.5298 105.3084)
+		(stroke
+			(width 0.1)
+			(type default)
+		)
+		(layer "F.SilkS")
+	)
+	(gr_line
+		(start 149.5298 108.5088)
+		(end 139.8778 108.5088)
+		(stroke
+			(width 0.1)
+			(type default)
+		)
+		(layer "F.SilkS")
+	)
+	(gr_line
+		(start 100.33 73.3044)
+		(end 100.33 55.5244)
+		(stroke
+			(width 0.1)
+			(type default)
+		)
+		(layer "F.SilkS")
+	)
+	(gr_line
+		(start 103.0986 55.5244)
+		(end 103.0986 59.6835)
+		(stroke
+			(width 0.1)
+			(type default)
+		)
+		(layer "F.SilkS")
+	)
+	(gr_line
+		(start 103.172 67.3635)
+		(end 103.172 73.279)
+		(stroke
+			(width 0.1)
+			(type default)
+		)
+		(layer "F.SilkS")
+	)
+	(gr_line
+		(start 167.3352 56.0578)
+		(end 167.3352 62.9412)
+		(stroke
+			(width 0.1)
+			(type default)
+		)
+		(layer "F.SilkS")
+	)
+	(gr_line
+		(start 100.33 69.469)
+		(end 103.2002 69.469)
+		(stroke
+			(width 0.1)
+			(type default)
+		)
+		(layer "F.SilkS")
+	)
+	(gr_line
+		(start 103.2002 65.4812)
+		(end 100.72 65.4812)
+		(stroke
+			(width 0.1)
+			(type default)
+		)
+		(layer "F.SilkS")
+	)
+	(gr_line
+		(start 103.172 73.279)
+		(end 100.33 73.279)
+		(stroke
+			(width 0.1)
+			(type default)
+		)
+		(layer "F.SilkS")
+	)
+	(gr_line
+		(start 100.33 55.5244)
+		(end 103.0986 55.5244)
+		(stroke
+			(width 0.1)
+			(type default)
+		)
+		(layer "F.SilkS")
+	)
+	(gr_line
+		(start 160.8328 59.4995)
+		(end 178.2064 59.4995)
+		(stroke
+			(width 0.1)
+			(type default)
+		)
+		(layer "F.SilkS")
+	)
+	(gr_line
+		(start 103.1494 60.7568)
+		(end 100.72 60.7568)
+		(stroke
+			(width 0.1)
+			(type default)
+		)
+		(layer "F.SilkS")
+	)
+	(gr_line
+		(start 160.8582 61.4172)
+		(end 178.2064 61.4172)
+		(stroke
+			(width 0.1)
+			(type default)
+		)
+		(layer "F.SilkS")
+	)
+	(gr_line
+		(start 160.8328 58.0136)
+		(end 178.2318 58.0136)
+		(stroke
+			(width 0.1)
+			(type default)
+		)
+		(layer "F.SilkS")
+	)
+	(gr_line
 		(start 151.511 94.75)
 		(end 205.58 94.75)
@@
 		)
 	)
-	(gr_text "RED"
-		(at 205.59395 68.843525 90)
+	(gr_text "SEL"
+		(at 101.6254 71.4756 0)
 		(layer "F.SilkS")
 		(effects
@@
 				(thickness 0.15)
 			)
-			(justify left bottom)
 		)
 	)
-	(gr_text "+5V"
-		(at 102.619175 66.8909 90)
+	(gr_text "RED"
+		(at 205.59395 68.843525 90)
 		(layer "F.SilkS")
 		(effects
@@
 		)
 	)
-	(gr_text "2"
-		(at 100.1903 69.402325 -90)
-		(layer "F.SilkS")
-		(effects
-			(font
-				(size 1 1)
-				(thickness 0.15)
-			)
-			(justify left bottom)
-		)
-	)
-	(gr_text "GND"
-		(at 102.6541 62.601475 90)
-		(layer "F.SilkS")
-		(effects
-			(font
-				(size 1 1)
-				(thickness 0.15)
-			)
-			(justify left bottom)
-		)
-	)
-	(gr_text_box "JKA1-1 JKA1-2\nI2CCLK  I2CDATA\nGND     3V3"
+	(gr_text_box "UPPER   LOWER\nJKA1-1  JKA1-2\nI2CCLK  I2CDATA\nGND       3V3"
 		(start 139.827732 103.2764)
-		(end 149.500148 109.519816)
+		(end 149.500148 110.2614)
 		(layer "F.SilkS")
 		(effects
@@
 				(thickness 0.1)
 			)
-			(justify left top)
+			(justify right top)
 		)
 		(border yes)
@@
 		)
 	)
-	(gr_text_box "SWITCH U3-40-PC9\nENC1   ENC2\nGND    5V"
+	(gr_text_box "UPPER   LOWER\nSWITCH U3-40-PC9\nENC1   ENC2\nGND    5V"
 		(locked yes)
 		(start 160.8328 56.1086)
