File: Gotek.kicad_sch (KiCad schematic)
At the start: 62 parts, among them J10 Conn_01x04_Pin, J3 Conn_01x03_Pin, J4 Conn_01x02_Pin, J5 Conn_01x02, J7 OLED, J8 RotaryEncoder, P1 2005280260, P3 USB_A, U3 AT32F435RGT7, U4 AMS1117-3.3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

Commit message: Add files via upload
Removed L3 Green LED and changed R21 to 12K to reduce it's brightness. Also increased the pad sizes for the diode D1D to make it easier to hand solder. Minor changes to silk screen.
Parts:
- L5: now fitted
- R21: value 1K -> 12K
Changed lines of the file:
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@@
 	(title_block
 		(title "Gotek(?) Handrawn Schematic, Layout and Gerbers")
-		(date "2025-02-20")
-		(rev "1.0")
+		(date "2025-04-11")
+		(rev "1.1")
 		(company "LiveBoxAndy")
 		(comment 1 "chip were removed to allow the routing underneath to be checked.")
 		(comment 2 "with the cable interface from an SFR1M44-DU26 (SFRC2D.B). The processor and the 74 ")
 		(comment 3 "Based on pictures and meter readings of an SRFKC30.AT4.35 for the processor bits mated")
-		(comment 4 "Correct JK1 and J8 Pin Idents. Point-Point wiring did not change.")
+		(comment 4 "Changed R21 to 12K to reduce brightness.")
 	)
 	(junction
@@
 			)
 		)
-		(property "Value" "1K"
+		(property "Value" "12K"
 			(at 255.778 119.38 90)
 			(effects
@@
 		(in_bom yes)
 		(on_board yes)
-		(dnp yes)
+		(dnp no)
 		(property "Reference" "L5"
 			(at 263.398 133.858 90)

Commit message: Minor Changes
Update for Kicad 9
Added ibom (bom/ibom.html)
Restructured folders.
Parts:
- C17, J10, J3, J4, JKA1, L3, U8: now fitted
Changed lines of the file:
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@@
 (kicad_sch
-	(version 20231120)
+	(version 20250114)
 	(generator "eeschema")
-	(generator_version "8.0")
+	(generator_version "9.0")
 	(paper "A4")
 	(title_block
@@
 		(comment 4 "Changed R21 to 12K to reduce brightness.")
 	)
+	(text "S1"
+		(exclude_from_sim no)
+		(at 122.682 88.392 0)
+		(effects
+			(font
+				(size 1.27 1.27)
+			)
+		)
+	)
+	(text "C16 is placed close\nto pins 31 & 32"
+		(exclude_from_sim no)
+		(at 228.346 143.51 0)
+		(effects
+			(font
+				(size 1.27 1.27)
+			)
+		)
+	)
 	(junction
 		(at 85.344 162.56)
@@
 		)
 	)
-	(text "S1"
-		(exclude_from_sim no)
-		(at 122.682 88.392 0)
-		(effects
-			(font
-				(size 1.27 1.27)
-			)
-		)
-	)
-	(text "C16 is placed close\nto pins 31 & 32"
-		(exclude_from_sim no)
-		(at 228.346 143.51 0)
-		(effects
-			(font
-				(size 1.27 1.27)
-			)
-		)
-	)
 	(label "I2C2_DTA"
 		(at 237.998 150.622 180)
@@
 		(in_bom yes)
 		(on_board yes)
-		(dnp yes)
+		(dnp no)
 		(property "Reference" "U8"
 			(at 249.174 22.352 0)
@@
 		(in_bom yes)
 		(on_board yes)
-		(dnp yes)
+		(dnp no)
 		(property "Reference" "JKA1"
 			(at 277.749 136.906 0)
@@
 		(in_bom yes)
 		(on_board yes)
-		(dnp yes)
+		(dnp no)
 		(property "Reference" "J3"
 			(at 129.794 184.15 0)
@@
 		(in_bom yes)
 		(on_board yes)
-		(dnp yes)
+		(dnp no)
 		(fields_autoplaced yes)
 		(property "Reference" "J10"
@@
 		(in_bom yes)
 		(on_board yes)
-		(dnp yes)
+		(dnp no)
 		(property "Reference" "J4"
 			(at 129.794 190.754 0)
@@
 		(in_bom yes)
 		(on_board yes)
-		(dnp yes)
+		(dnp no)
 		(property "Reference" "C17"
 			(at 139.954 35.306 0)
@@
 		(in_bom yes)
 		(on_board yes)
-		(dnp yes)
+		(dnp no)
 		(property "Reference" "L3"
 			(at 271.526 134.366 90)
@@
 		(at 65.278 189.738)
 		(size 14.986 3.81)
+		(exclude_from_sim no)
+		(in_bom yes)
+		(on_board yes)
+		(dnp no)
 		(fields_autoplaced yes)
 		(stroke
@@
 		)
 	)
+	(embedded_fonts no)
 )
